File: PCB Version 0.6/gyro.kicad_sch (KiCad schematic)
At the start: 7 parts, among them U12 ICM-42688-P

Commit message: wip layout
Parts:
- removed R38, R39, R40: 22, Resistor_SMD:R_0402_1005Metric, symbol Device:R
Connections:
- net SPI0.MISO: now also U12.1 (SDO)
- net SPI0.MOSI: now also U12.14 (SDx)
- net SPI0.SCLK: now also U12.13 (SCx)

Commit message: wip routing
Connections:
- no-connect marks 0 -> 4
Changed lines of the file:
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@@
 		(color 0 0 0 0)
+	)
+	(no_connect
+		(at 107.95 58.42)
+	)
+	(no_connect
+		(at 107.95 55.88)
+	)
+	(no_connect
+		(at 107.95 53.34)
+	)
+	(no_connect
+		(at 107.95 50.8)
 	)
 	(bus_entry
