File: PCB Version 0.6/Kolibri v0.6.kicad_pcb (KiCad board)
At the start: 8 copper layers, 28 x 28 mm, 199 parts, among them IC1 SX1280IMLTRT, IC5 LMR38025SDRRR, IC6 LMR38025SDRRR, J1 USB_C_Receptacle_USB2.0_16P, J3 Conn_Coaxial_Small, J5 Conn_01x08_MountingPin, J6 Conn_01x06_MountingPin, J7 Conn_01x06_MountingPin, Q1 BSS138, U1 RP2350A, U10 W25Q16JVUXIQ, U11 LPS22HB, U12 ICM-42688-P, U2 C5250982, U3 ESP32-C3, U4 TPS2116DRL, U5 AT7456E, U6 MT29F2G01ABAGDWB-IT:G, U7 TPS746-3.3DRV, U8 LMV321, Y1 Crystal_GND24, Y2 Crystal_GND24, Y4 Crystal_GND24, Y5 Crystal_GND24

Commit message: wip layout
Parts:
- removed C82: 1u, Capacitor_SMD:C_0402_1005Metric
- removed D18: orange, LED_SMD:LED_0603_1608Metric
- removed P19: ~, Kolibri custom:Solder_Pad_rounded_dual
- removed R32, R38, R39, R40: 22, Resistor_SMD:R_0402_1005Metric
- added P5: ~, Kolibri custom:Solder_Pad_rounded, F.Cu at (101.3, 82.0)
- C14: moved to F.Cu
- C16, C28, C40, C41, C44, C45, C48, C65, C66, C71, C72, C84, C88, D1, D10, D11, D15, IC6, J6, J7, L5, L7, P1, P10, P11, P12, P13, P14, P15, P16, P17, P2, P20, P21, P22, P23, P24, P28, P29, P3, P30, P34, P35, P36, P4, Q1, R10, R13, R14, R17, R19, R20, R29, R31, R33, R34, R35, R36, R37, R8, U8: moved to B.Cu
- C63, C64: footprint Capacitor_SMD:C_0603_1608Metric -> Capacitor_SMD:C_0402_1005Metric; moved to B.Cu
- C68: value 2.2u -> 4.7u; footprint Capacitor_SMD:C_1206_3216Metric -> Capacitor_SMD:C_0805_2012Metric
- C69: value 2.2u -> 4.7u; footprint Capacitor_SMD:C_1206_3216Metric -> Capacitor_SMD:C_0805_2012Metric; moved to B.Cu
- P18: footprint Kolibri custom:Solder_Pad_rounded_dual -> Kolibri custom:Solder_Pad_rounded
- U7: footprint Package_SON:WSON-6-1EP_2x2mm_P0.65mm_EP1x1.6mm_ThermalVias -> Package_SON:WSON-6-1EP_2x2mm_P0.65mm_EP1x1.6mm; moved to B.Cu
- moved R29 161.4 mm to (87.2, 104.6), turned to 180 degrees
- moved R30 160.2 mm to (89.9, 114.2), turned to 180 degrees
- moved D16 158.5 mm to (87.4, 114.0)
- moved D15 158.1 mm to (86.8, 106.5), turned to 90 degrees
- moved R31 148.1 mm to (106.2, 113.3)
- moved C16 147.7 mm to (97.6, 94.0), turned to -90 degrees
- moved D1 146.9 mm to (98.3, 91.7), turned to -90 degrees
- moved C46 143.6 mm to (103.8, 99.0)
- moved R41 143.3 mm to (105.7, 99.0)
- moved U6 142.4 mm to (107.5, 95.3), turned to 180 degrees
- moved D17 139.5 mm to (106.0, 112.5), turned to -90 degrees
- moved C17 135.1 mm to (110.9, 77.6)
- moved C18 135.1 mm to (104.6, 75.6)
- moved C19 135.1 mm to (104.6, 77.6)
- moved C20 135.1 mm to (104.6, 79.6)
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Connections:
- C31 pad 1: +3V3_ELRS -> +3V3
- C84 pad 1: +3V3_ELRS -> +3V3
- P18 pad 1: /Video.In -> /Video.Out
- U12 pad 1: Net-(U12-SDO) -> /SPI0.MISO
- U12 pad 13: Net-(U12-SCx) -> /SPI0.SCLK
- U12 pad 14: Net-(U12-SDx) -> /SPI0.MOSI
- U7 pad 1: +3V3_ELRS -> +3V3
Other:
- outline, holes or cut-outs redrawn

Commit message: wip layout
Parts:
- removed P30: ~, Kolibri custom:Solder_Pad_octa_dual
- added P19: ~, Kolibri custom:Solder_Pad_rounded, F.Cu at (100.0, 87.0)
- P10, P11, P16, P17: moved to F.Cu
- P20, P21: footprint Kolibri custom:Solder_Pad_rounded_dual -> Kolibri custom:Solder_Pad_rounded; moved to F.Cu
- P22: footprint Kolibri custom:Solder_Pad_rounded_dual -> Kolibri custom:Solder_Pad_rect; moved to F.Cu
- P25: footprint Kolibri custom:Solder_Pad_rect_dual -> Kolibri custom:Solder_Pad_octa
- P29: footprint Kolibri custom:Solder_Pad_octa_dual -> Kolibri custom:Solder_Pad_octa; moved to F.Cu
- moved P16 34.4 mm to (92.5, 111.4), turned to 0 degrees
- moved P17 32.0 mm to (93.4, 109.5), turned to 0 degrees
- moved P23 31.9 mm to (90.7, 87.0)
- moved P28 31.1 mm to (109.0, 87.0)
- moved R30 28.4 mm to (103.4, 89.2), turned to 90 degrees
- moved D16 28.4 mm to (102.2, 89.8), turned to 90 degrees
- moved P20 23.1 mm to (98.2, 87.0), turned to 0 degrees
- moved P10 20.9 mm to (105.4, 87.0), turned to 0 degrees
- moved P25 20.6 mm to (92.5, 87.0)
- moved P11 19.1 mm to (105.4, 88.8), turned to 0 degrees
- moved P22 15.7 mm to (107.2, 87.0), turned to 0 degrees
- moved P21 14.5 mm to (118.1, 77.7), turned to 0 degrees
- moved P29 12.9 mm to (107.2, 88.8), turned to 0 degrees
- moved P5 5.55 mm to (103.6, 87.0)
- moved P18 2.89 mm to (101.8, 87.0)
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Connections:
- P20 pad 1: /Connectors/LED -> /Spk.-
- P21 pad 1: /Spk.+ -> /Connectors/LED
- P22 pad 1: /Spk.- -> GND
- P25 pad 1: GND -> +5V

Commit message: layout first draft done
Parts:
- added P30: ~, Kolibri custom:Solder_Pad_octa, F.Cu at (111.0, 106.6)
- added P37: ~, Kolibri custom:Solder_Pad_rounded, B.Cu at (89.2, 113.2)
- added P38: ~, Kolibri custom:Solder_Pad_rounded, F.Cu at (113.0, 106.6)
- added P39: ~, Kolibri custom:Solder_Pad_octa, F.Cu at (113.0, 98.0)
- added P40: ~, Kolibri custom:Solder_Pad_rect, F.Cu at (106.5, 113.0)
- added P41: ~, Kolibri custom:Solder_Pad_octa, B.Cu at (91.2, 113.2)
- added P42: ~, Kolibri custom:Solder_Pad_rect, B.Cu at (86.8, 110.4)
- added P43: ~, Kolibri custom:Solder_Pad_rect, B.Cu at (86.6, 89.2)
- C17, C18, C19, C20, D14, D17, P21, R28: moved to B.Cu
- P23, P24: footprint Kolibri custom:Solder_Pad_rect_dual -> Kolibri custom:Solder_Pad_rect; moved to F.Cu
- P28, P34: footprint Kolibri custom:Solder_Pad_octa_dual -> Kolibri custom:Solder_Pad_octa; moved to F.Cu
- P33: footprint Kolibri custom:Solder_Pad_octa_dual -> Kolibri custom:Solder_Pad_octa
- moved D5 42.8 mm to (90.2, 113.4), turned to 180 degrees
- moved D4 37.2 mm to (86.6, 109.8), turned to 90 degrees
- moved C19 35.7 mm to (86.8, 108.5)
- moved D6 34.2 mm to (109.8, 113.4), turned to 180 degrees
- moved C20 33.9 mm to (106.5, 113.4), turned to 180 degrees
- moved D7 32.7 mm to (113.4, 109.8), turned to -90 degrees
- moved D17 30.5 mm to (90.4, 86.2), turned to 180 degrees
- moved R31 30.1 mm to (90.8, 87.5), turned to 180 degrees
- moved C17 27.5 mm to (86.8, 90.8), turned to 180 degrees
- moved D3 23.1 mm to (86.6, 90.2), turned to -90 degrees
- moved D2 19.7 mm to (90.2, 86.6)
- moved R28 16.1 mm to (114.0, 90.1), turned to 90 degrees
- moved D14 15.8 mm to (112.8, 89.8), turned to 90 degrees
- moved D8 14.0 mm to (113.4, 90.2), turned to -90 degrees
- moved P31 13.6 mm to (87.0, 107.4)
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Connections:
- net /ELRS/GPIO10 renamed /PWM.1
- net /ELRS/GPIO18 renamed /PWM.2
- P34 pad 1: +3V3 -> +10V
Other:
- board size 28 x 28 mm -> 29.4 x 29.4 mm

Commit message: wip routing
Parts:
- C28: moved to F.Cu
- U8: value LMV321 -> C3029047
- moved C28 2.56 mm to (93.6, 102.5), turned to 90 degrees
- moved P8 1.90 mm to (86.9, 95.9)
- moved P9 1.70 mm to (86.9, 97.7)
- moved C16 0.40 mm to (97.6, 94.3)
- moved P37 0.40 mm to (89.2, 113.6)
- moved P14 0.39 mm to (96.9, 96.0)
- moved C69 0.35 mm to (96.3, 105.1)
- moved P41 0.30 mm to (91.2, 113.5)
- moved P42 0.30 mm to (86.5, 110.4)
- moved C44 0.25 mm to (92.9, 101.5)
- moved P43 0.22 mm to (86.5, 89.0)
- moved P21 0.20 mm to (110.8, 86.4)
- moved C12 0.15 mm to (98.8, 90.1)
- moved C13 0.15 mm to (98.8, 91.0)
- moved P40 0.11 mm to (106.5, 113.1)
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Connections:
- C44 pad 1: +3V3_ELRS -> +3V3
- C45 pad 1: +3V3_ELRS -> +3V3
- IC1 pad 11: +3V3_ELRS -> +3V3
- IC1 pad 15: +3V3_ELRS -> +3V3
- J6 pad 5: /I2C0.SDA -> /I2C0.SCL
- J6 pad 6: /I2C0.SCL -> /I2C0.SDA
Routing:
- net /I2C0.SDA: track 0.00 -> 50.5 mm, vias 0 -> 4
- net /I2C0.SCL: track 0.00 -> 40.8 mm, vias 0 -> 4
- net /SPI0.MOSI: track 0.00 -> 40.2 mm, vias 0 -> 2
- net /SPI0.SCLK: track 0.00 -> 40.0 mm, vias 0 -> 2
- net /ELRS/WIFI_ANTENNA: track 0.00 -> 38.7 mm, vias 0 -> 1
- net /SPI0.MISO: track 0.00 -> 35.3 mm, vias 0 -> 2
- net Net-(U1-USB_DM): track 0.00 -> 29.8 mm, vias 0 -> 2
- net Net-(U1-USB_DP): track 0.00 -> 29.6 mm, vias 0 -> 2
- net /USB.D-: track 0.00 -> 27.7 mm, vias 0 -> 2
- net /USB.D+: track 0.00 -> 27.4 mm, vias 0 -> 2
- net GND: track 0.00 -> 27.1 mm, vias 0 -> 6
- net +3V3: track 0.00 -> 26.1 mm, vias 0 -> 13
- net /RP2350/Gyro_SS: track 0.00 -> 25.6 mm, vias 0 -> 2
- net /U0.TX: track 0.00 -> 25.5 mm, vias 0 -> 2
- net /U0.RX: track 0.00 -> 23.0 mm, vias 0 -> 3
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- added copper zone on F.Cu, net +1V1
- added copper zone on B.Cu, net +5V_BUCK
- added copper zone on B.Cu, net Net-(IC5-SW_1)
- added copper zone on F.Cu, net Net-(IC5-SW_1)
- added copper zone on B.Cu, net Net-(IC6-SW_1)
- added copper zone on F.Cu, net Net-(IC6-SW_1)
- added copper zone on B.Cu, net VCC
- added copper zone on F.Cu, net VCC

Commit message: wip
Parts:
- moved C69 0.05 mm to (96.3, 105.2)
Connections:
- C81 pad 2: Net-(U2-GND) -> GND
- C88 pad 2: Net-(U2-GND) -> GND
- P37 pad 1: /Connectors/PWM.1 -> /PWM.2
- P38 pad 1: /Connectors/PWM.2 -> /PWM.1
- U2 pad 1: Net-(U2-GND) -> GND
Routing:
- net +4V5: track 1.70 -> 35.7 mm, vias 0 -> 3
- net GND: track 27.1 -> 55.2 mm, vias 6 -> 63
- net Net-(R33-Pad2): track 0.00 -> 24.2 mm, vias 0 -> 2
- net /PWM.1: track 0.13 -> 20.3 mm, vias 1 -> 2
- net /U2.TX: track 5.91 -> 25.5 mm
- net /RP2350/Speaker: track 3.81 -> 23.3 mm, vias 1 -> 2
- net /U2.RX: track 3.81 -> 21.9 mm
- net /Motor.4: track 17.1 -> 33.3 mm, vias 2 -> 3
- net /Motor.3: track 18.6 -> 33.9 mm, vias 2 -> 3
- net +3V3: track 26.1 -> 39.1 mm, vias 13 -> 19
- net /ADC/VBat_ADC: track 1.92 -> 14.1 mm, vias 1 -> 2
- net /Motor.1: track 16.1 -> 28.2 mm, vias 2 -> 3
- net /Motor.2: track 17.5 -> 29.1 mm, vias 2 -> 3
- net Net-(D1-DOUT): track 0.00 -> 10.6 mm, vias 0 -> 1
- net /PWM.2: track 0.00 -> 9.75 mm, vias 1 -> 2
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- added copper zone on In2.Cu, net +1V1
- added copper zone on In3.Cu, net +3V3
- added copper zone on B.Cu, net GND
- added copper zone on F.Cu, net GND
- added copper zone on In1.Cu, net GND
- added copper zone on In2.Cu, net GND
- added copper zone on In4.Cu, net GND
- added copper zone on In5.Cu, net GND
