File: PCB Version 0.6/ELRS.kicad_sch (KiCad schematic)
At the start: 32 parts, among them IC1 SX1280IMLTRT, J3 Conn_Coaxial_Small, U3 ESP32-C3, Y2 Crystal_GND24, Y5 Crystal_GND24

Commit message: WIP layout
Parts:
- C26: footprint (none) -> Capacitor_SMD:C_0402_1005Metric
- C33, C34, C36, C37, C38, C39, C40, C41, C42, C43, C44, C45: footprint Capacitor_SMD:C_0402_1005Metric_Pad0.74x0.62mm_HandSolder -> Capacitor_SMD:C_0402_1005Metric
- L2: footprint Inductor_SMD:L_0402_1005Metric_Pad0.77x0.64mm_HandSolder -> Inductor_SMD:L_0402_1005Metric
Connections:
- net +3V3: now also C34.1, C36.1, L2.1
- net +3V3_ELRS: no longer C34.1, C36.1, L2.1
Changed lines of the file:
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@@
 	)
 	(junction
-		(at 88.9 92.71)
-		(diameter 0)
-		(color 0 0 0 0)
-	)
-	(junction
 		(at 41.91 152.4)
 		(diameter 0)
@@
 	)
 	(junction
+		(at 88.9 92.71)
+		(diameter 0)
+		(color 0 0 0 0)
+	)
+	(junction
 		(at 184.15 196.85)
 		(diameter 0)
@@
 	)
 	(symbol
-		(lib_id "power:+3V3")
-		(at 88.9 92.71 0)
-		(unit 1)
-		(exclude_from_sim no)
-		(in_bom yes)
-		(on_board yes)
-		(dnp no)
-		(property "Reference" "#PWR39"
-			(at 88.9 96.52 0)
-			(effects
-				(font
-					(size 1.27 1.27)
-				)
-				(hide yes)
-			)
-		)
-		(property "Value" "+3V3_ELRS"
-			(at 83.566 88.392 0)
-			(effects
-				(font
-					(size 1.27 1.27)
-				)
-				(justify left)
-			)
-		)
-		(property "Footprint" ""
-			(at 88.9 92.71 0)
-			(effects
-				(font
-					(size 1.27 1.27)
-				)
-				(hide yes)
-			)
-		)
-		(property "Datasheet" ""
-			(at 88.9 92.71 0)
-			(effects
-				(font
-					(size 1.27 1.27)
-				)
-				(hide yes)
-			)
-		)
-		(property "Description" "Power symbol creates a global label with name \"+3V3\""
-			(at 88.9 92.71 0)
-			(effects
-				(font
-					(size 1.27 1.27)
-				)
-				(hide yes)
-			)
-		)
-		(pin "1"
-		)
-		(instances
-			(project "Kolibri v0.6"
-				(path "/1651f454-30c0-48ea-9fcf-6c96a661786a/f86b6c62-cfc0-4383-b218-cc390d004fb8"
-					(reference "#PWR39")
-					(unit 1)
-				)
-			)
-		)
-	)
-	(symbol
 		(lib_id "Device:R")
 		(at 215.9 113.03 0)
@@
 			)
 		)
-		(property "Footprint" "Capacitor_SMD:C_0402_1005Metric_Pad0.74x0.62mm_HandSolder"
+		(property "Footprint" "Capacitor_SMD:C_0402_1005Metric"
 			(at 178.7652 102.87 0)
 			(effects
@@
 			)
 		)
-		(property "Footprint" "Inductor_SMD:L_0402_1005Metric_Pad0.77x0.64mm_HandSolder"
+		(property "Footprint" "Inductor_SMD:L_0402_1005Metric"
 			(at 113.03 92.71 0)
 			(effects
@@
 			)
 		)
-		(property "Footprint" "Capacitor_SMD:C_0402_1005Metric_Pad0.74x0.62mm_HandSolder"
+		(property "Footprint" "Capacitor_SMD:C_0402_1005Metric"
 			(at 102.5652 100.33 0)
 			(effects
@@
 			)
 		)
-		(property "Footprint" ""
+		(property "Footprint" "Capacitor_SMD:C_0402_1005Metric"
 			(at 177.4952 78.74 0)
 			(effects
@@
 			)
 		)
-		(property "Footprint" "Capacitor_SMD:C_0402_1005Metric_Pad0.74x0.62mm_HandSolder"
+		(property "Footprint" "Capacitor_SMD:C_0402_1005Metric"
 			(at 316.5348 193.04 0)
 			(effects
@@
 			)
 		)
-		(property "Footprint" "Capacitor_SMD:C_0402_1005Metric_Pad0.74x0.62mm_HandSolder"
+		(property "Footprint" "Capacitor_SMD:C_0402_1005Metric"
 			(at 279.4 198.4248 0)
 			(effects
@@
 			)
 		)
-		(property "Footprint" "Capacitor_SMD:C_0402_1005Metric_Pad0.74x0.62mm_HandSolder"
+		(property "Footprint" "Capacitor_SMD:C_0402_1005Metric"
 			(at 102.5652 199.39 0)
 			(effects
@@
 			)
 		)
-		(property "Footprint" "Capacitor_SMD:C_0402_1005Metric_Pad0.74x0.62mm_HandSolder"
+		(property "Footprint" "Capacitor_SMD:C_0402_1005Metric"
 			(at 55.88 143.8148 0)
 			(effects
@@
 	)
 	(symbol
+		(lib_id "power:+3V3")
+		(at 88.9 92.71 0)
+		(unit 1)
+		(exclude_from_sim no)
+		(in_bom yes)
+		(on_board yes)
+		(dnp no)
+		(fields_autoplaced yes)
+		(property "Reference" "#PWR039"
+			(at 88.9 96.52 0)
+			(effects
+				(font
+					(size 1.27 1.27)
+				)
+				(hide yes)
+			)
+		)
+		(property "Value" "+3V3"
+			(at 88.9 87.63 0)
+			(effects
+				(font
+					(size 1.27 1.27)
+				)
+			)
+		)
+		(property "Footprint" ""
+			(at 88.9 92.71 0)
+			(effects
+				(font
+					(size 1.27 1.27)
+				)
+				(hide yes)
+			)
+		)
+		(property "Datasheet" ""
+			(at 88.9 92.71 0)
+			(effects
+				(font
+					(size 1.27 1.27)
+				)
+				(hide yes)
+			)
+		)
+		(property "Description" "Power symbol creates a global label with name \"+3V3\""
+			(at 88.9 92.71 0)
+			(effects
+				(font
+					(size 1.27 1.27)
+				)
+				(hide yes)
+			)
+		)
+		(pin "1"
+		)
+		(instances
+			(project ""
+				(path "/1651f454-30c0-48ea-9fcf-6c96a661786a/f86b6c62-cfc0-4383-b218-cc390d004fb8"
+					(reference "#PWR039")
+					(unit 1)
+				)
+			)
+		)
+	)
+	(symbol
 		(lib_id "SamacSys_Parts:SX1280IMLTRT")
 		(at 283.21 160.02 0)
@@
 			)
 		)
-		(property "Footprint" "Capacitor_SMD:C_0402_1005Metric_Pad0.74x0.62mm_HandSolder"
+		(property "Footprint" "Capacitor_SMD:C_0402_1005Metric"
 			(at 266.7 160.9852 0)
 			(effects
@@
 			)
 		)
-		(property "Footprint" "Capacitor_SMD:C_0402_1005Metric_Pad0.74x0.62mm_HandSolder"
+		(property "Footprint" "Capacitor_SMD:C_0402_1005Metric"
 			(at 120.3452 100.33 0)
 			(effects
@@
 			)
 		)
-		(property "Footprint" "Capacitor_SMD:C_0402_1005Metric_Pad0.74x0.62mm_HandSolder"
+		(property "Footprint" "Capacitor_SMD:C_0402_1005Metric"
 			(at 55.88 151.4348 0)
 			(effects
@@
 			)
 		)
-		(property "Footprint" "Capacitor_SMD:C_0402_1005Metric_Pad0.74x0.62mm_HandSolder"
+		(property "Footprint" "Capacitor_SMD:C_0402_1005Metric"
 			(at 341.3252 175.26 0)
 			(effects
@@
 			)
 		)
-		(property "Footprint" "Capacitor_SMD:C_0402_1005Metric_Pad0.74x0.62mm_HandSolder"
+		(property "Footprint" "Capacitor_SMD:C_0402_1005Metric"
 			(at 89.8652 100.33 0)
 			(effects
@@
 			)
 		)
-		(property "Footprint" "Capacitor_SMD:C_0402_1005Metric_Pad0.74x0.62mm_HandSolder"
+		(property "Footprint" "Capacitor_SMD:C_0402_1005Metric"
 			(at 304.4952 205.74 0)
 			(effects

Commit message: layout first draft done
Connections:
- net GPIO10 renamed PWM.1
- net GPIO18 renamed PWM.2
Changed lines of the file:
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@@
+		)
+	)
+	(bus_entry
+		(at 101.6 121.92)
+		(size 2.54 2.54)
+		(stroke
+			(width 0)
+			(type default)
+		)
+	)
+	(bus_entry
+		(at 101.6 119.38)
+		(size 2.54 2.54)
+		(stroke
+			(width 0)
+			(type default)
 		)
 	)
@@
 		)
 	)
+	(bus
+		(pts
+			(xy 101.6 121.92) (xy 101.6 119.38)
+		)
+		(stroke
+			(width 0)
+			(type default)
+		)
+	)
 	(wire
 		(pts
@@
 		(pts
 			(xy 327.66 220.98) (xy 327.66 193.04)
+		)
+		(stroke
+			(width 0)
+			(type default)
+		)
+	)
+	(bus
+		(pts
+			(xy 74.93 119.38) (xy 101.6 119.38)
 		)
 		(stroke
@@
 		)
 	)
-	(label "GPIO18"
-		(at 104.14 124.46 0)
+	(label "PWM.1"
+		(at 104.14 121.92 0)
 		(effects
 			(font
@@
 		)
 	)
-	(label "GPIO10"
-		(at 104.14 121.92 0)
-		(effects
-			(font
-				(size 1.27 1.27)
-			)
-			(justify left bottom)
-		)
-	)
 	(label "U0{TX RX}"
 		(at 71.12 137.16 180)
@@
 		)
 	)
+	(label "PWM.2"
+		(at 104.14 124.46 0)
+		(effects
+			(font
+				(size 1.27 1.27)
+			)
+			(justify left bottom)
+		)
+	)
 	(label "RADIO_BUSY"
 		(at 104.14 114.3 0)
@@
 		)
 	)
+	(label "PWM{[1..2]}"
+		(at 81.28 119.38 0)
+		(effects
+			(font
+				(size 1.27 1.27)
+			)
+			(justify left bottom)
+		)
+	)
 	(label "ELRS_LED_RGB"
 		(at 60.96 195.58 0)
@@
 		)
 	)
+	(hierarchical_label "PWM"
+		(shape output)
+		(at 74.93 119.38 180)
+		(effects
+			(font
+				(size 1.27 1.27)
+			)
+			(justify right)
+		)
+	)

Commit message: wip routing
Connections:
- net +3V3_ELRS is gone; now on net +3V3: C44.1, C45.1, IC1.11 (VBAT_IO), IC1.15 (VBAT)
Changed lines of the file:
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@@
 	)
 	(junction
-		(at 303.53 195.58)
+		(at 88.9 100.33)
 		(diameter 0)
 		(color 0 0 0 0)
 	)
 	(junction
-		(at 88.9 100.33)
+		(at 121.92 78.74)
 		(diameter 0)
 		(color 0 0 0 0)
 	)
 	(junction
-		(at 121.92 78.74)
+		(at 303.53 198.12)
+		(diameter 0)
+		(color 0 0 0 0)
+	)
+	(junction
+		(at 340.36 167.64)
 		(diameter 0)
 		(color 0 0 0 0)
@@
 	)
 	(junction
-		(at 340.36 167.64)
-		(diameter 0)
-		(color 0 0 0 0)
-	)
-	(junction
 		(at 279.4 199.39)
 		(diameter 0)
@@
 	(wire
 		(pts
-			(xy 303.53 193.04) (xy 303.53 195.58)
-		)
-		(stroke
-			(width 0)
-			(type default)
-		)
-	)
-	(wire
-		(pts
 			(xy 318.77 160.02) (xy 334.01 160.02)
 		)
@@
 	(wire
 		(pts
-			(xy 303.53 195.58) (xy 303.53 198.12)
+			(xy 303.53 193.04) (xy 303.53 198.12)
 		)
 		(stroke
@@
 		(on_board yes)
 		(dnp no)
-		(fields_autoplaced yes)
 		(property "Reference" "C34"
 			(at 105.41 95.2499 0)
@@
 	)
 	(symbol
+		(lib_id "power:+3V3")
+		(at 303.53 198.12 270)
+		(unit 1)
+		(exclude_from_sim no)
+		(in_bom yes)
+		(on_board yes)
+		(dnp no)
+		(fields_autoplaced yes)
+		(property "Reference" "#PWR061"
+			(at 299.72 198.12 0)
+			(effects
+				(font
+					(size 1.27 1.27)
+				)
+				(hide yes)
+			)
+		)
+		(property "Value" "+3V3"
+			(at 307.34 198.1199 90)
+			(effects
+				(font
+					(size 1.27 1.27)
+				)
+				(justify left)
+			)
+		)
+		(property "Footprint" ""
+			(at 303.53 198.12 0)
+			(effects
+				(font
+					(size 1.27 1.27)
+				)
+				(hide yes)
+			)
+		)
+		(property "Datasheet" ""
+			(at 303.53 198.12 0)
+			(effects
+				(font
+					(size 1.27 1.27)
+				)
+				(hide yes)
+			)
+		)
+		(property "Description" "Power symbol creates a global label with name \"+3V3\""
+			(at 303.53 198.12 0)
+			(effects
+				(font
+					(size 1.27 1.27)
+				)
+				(hide yes)
+			)
+		)
+		(pin "1"
+		)
+		(instances
+			(project ""
+				(path "/1651f454-30c0-48ea-9fcf-6c96a661786a/f86b6c62-cfc0-4383-b218-cc390d004fb8"
+					(reference "#PWR061")
+					(unit 1)
+				)
+			)
+		)
+	)
+	(symbol
 		(lib_id "Device:C")
 		(at 176.53 74.93 0)
@@
 	)
 	(symbol
+		(lib_id "power:+3V3")
+		(at 340.36 167.64 0)
+		(unit 1)
+		(exclude_from_sim no)
+		(in_bom yes)
+		(on_board yes)
+		(dnp no)
+		(fields_autoplaced yes)
+		(property "Reference" "#PWR058"
+			(at 340.36 171.45 0)
+			(effects
+				(font
+					(size 1.27 1.27)
+				)
+				(hide yes)
+			)
+		)
+		(property "Value" "+3V3"
+			(at 340.36 162.56 0)
+			(effects
+				(font
+					(size 1.27 1.27)
+				)
+			)
+		)
+		(property "Footprint" ""
+			(at 340.36 167.64 0)
+			(effects
+				(font
+					(size 1.27 1.27)
+				)
+				(hide yes)
+			)
+		)
+		(property "Datasheet" ""
+			(at 340.36 167.64 0)
+			(effects
+				(font
+					(size 1.27 1.27)
+				)
+				(hide yes)
+			)
+		)
+		(property "Description" "Power symbol creates a global label with name \"+3V3\""
+			(at 340.36 167.64 0)
+			(effects
+				(font
+					(size 1.27 1.27)
+				)
+				(hide yes)
+			)
+		)
+		(pin "1"
+		)
+		(instances
+			(project ""
+				(path "/1651f454-30c0-48ea-9fcf-6c96a661786a/f86b6c62-cfc0-4383-b218-cc390d004fb8"
+					(reference "#PWR058")
+					(unit 1)
+				)
+			)
+		)
+	)
+	(symbol
 		(lib_id "power:GND")
 		(at 247.65 179.07 0)
@@
 					(unit 1)
 				)
-			)
-		)
-	)
-	(symbol
-		(lib_id "power:+3V3")
-		(at 303.53 195.58 270)
-		(unit 1)
-		(exclude_from_sim no)
-		(in_bom yes)
-		(on_board yes)
-		(dnp no)
-		(property "Reference" "#PWR61"
-			(at 299.72 195.58 0)
-			(effects
-				(font
-					(size 1.27 1.27)
-				)
-				(hide yes)
-			)
-		)
-		(property "Value" "+3V3_ELRS"
-			(at 303.784 197.612 90)
-			(effects
-				(font
-					(size 1.27 1.27)
-				)
-				(justify left)
-			)
-		)
-		(property "Footprint" ""
-			(at 303.53 195.58 0)
-			(effects
-				(font
-					(size 1.27 1.27)
-				)
-				(hide yes)
-			)
-		)
-		(property "Datasheet" ""
-			(at 303.53 195.58 0)
-			(effects
-				(font
-					(size 1.27 1.27)
-				)
-				(hide yes)
-			)
-		)
-		(property "Description" "Power symbol creates a global label with name \"+3V3\""
-			(at 303.53 195.58 0)
-			(effects
-				(font
-					(size 1.27 1.27)
-				)
-				(hide yes)
-			)
-		)
-		(pin "1"
-		)
-		(instances
-			(project "Kolibri v0.5"
-				(path "/1651f454-30c0-48ea-9fcf-6c96a661786a/f86b6c62-cfc0-4383-b218-cc390d004fb8"
-					(reference "#PWR61")
-					(unit 1)
-				)
-			)
-		)
-	)
-	(symbol
-		(lib_id "power:+3V3")
-		(at 340.36 167.64 0)
-		(unit 1)
-		(exclude_from_sim no)
-		(in_bom yes)
-		(on_board yes)
-		(dnp no)
-		(property "Reference" "#PWR58"
-			(at 340.36 171.45 0)
-			(effects
-				(font
-					(size 1.27 1.27)
-				)
-				(hide yes)
-			)
-		)
-		(property "Value" "+3V3_ELRS"
-			(at 335.026 163.322 0)
-			(effects
-				(font
-					(size 1.27 1.27)
-				)
-				(justify left)
-			)
-		)
-		(property "Footprint" ""
-			(at 340.36 167.64 0)
-			(effects
-				(font
-					(size 1.27 1.27)
-				)
-				(hide yes)
-			)
-		)
-		(property "Datasheet" ""
-			(at 340.36 167.64 0)
-			(effects
-				(font
-					(size 1.27 1.27)
-				)
-				(hide yes)
-			)
-		)
-		(property "Description" "Power symbol creates a global label with name \"+3V3\""
-			(at 340.36 167.64 0)
-			(effects
-				(font
-					(size 1.27 1.27)
-				)
-				(hide yes)
-			)
-		)
-		(pin "1"
-		)
-		(instances
-			(project "Kolibri v0.5"
-				(path "/1651f454-30c0-48ea-9fcf-6c96a661786a/f86b6c62-cfc0-4383-b218-cc390d004fb8"
-					(reference "#PWR58")
-					(unit 1)
-				)

Commit message: ESP8685
Parts:
- removed U3: ESP32-C3, Package_DFN_QFN:QFN-32-1EP_5x5mm_P0.5mm_EP3.7x3.7mm, symbol MCU_Espressif:ESP32-C3
- added U3: ESP8685-H4, Package_DFN_QFN:QFN-28-1EP_4x4mm_P0.4mm_EP2.4x2.4mm, symbol Kolibri custom:ESP8685-H4
Connections:
- net +3V3: now also U3.11 (VDD3P3_RTC), U3.17 (VDD3P3_CPU), U3.18 (VDD_SPI), U3.27 (VDDA), U3.28 (VDDA)
- net ELRS_BUTTON: now also U3.15 (GPIO9)
- net ELRS_LED_RGB: now also U3.14 (GPIO8)
- net GND: now also U3.29 (GND)
- net GPIO0: now also U3.4 (XTAL_32K_P)
- net GPIO19: now also U3.22 (GPIO19)
- net PWM.1: now also U3.16 (GPIO10)
- net PWM.2: now also U3.21 (GPIO18)
- net RADIO_BUSY: now also U3.8 (GPIO3)
- net RADIO_DIO1: now also U3.5 (XTAL_32K_N)
- net RADIO_MISO: now also U3.10 (MTDI)
- net RADIO_MOSI: now also U3.9 (MTMS)
- net RADIO_NSS: now also U3.13 (MTDO)
- net RADIO_RST: now also U3.6 (GPIO2)
- net RADIO_SCK: now also U3.12 (MTCK)
- net U0.RX: now also U3.24 (U0TXD)
- net U0.TX: now also U3.23 (U0RXD)
- net at C35.1, R9.2: now also U3.7 (CHIP_EN)
- net at C37.1, L3.1: now also U3.1 (LNA_IN)
- net at L4.2: now also U3.26 (XTAL_P)
- net at C33.1, L2.2: now also U3.2 (VDD3P3), U3.3 (VDD3P3)
- net at C38.2, Y2.3: now also U3.25 (XTAL_N)
- no-connect marks 9 -> 5
Changed lines of the file:
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@@
 	)
 	(junction
-		(at 142.24 106.68)
+		(at 147.32 106.68)
 		(diameter 0)
 		(color 0 0 0 0)
@@
 	)
 	(junction
-		(at 147.32 106.68)
-		(diameter 0)
-		(color 0 0 0 0)
-	)
-	(junction
 		(at 298.45 124.46)
 		(diameter 0)
@@
 	)
 	(junction
+		(at 142.24 106.68)
+		(diameter 0)
+		(color 0 0 0 0)
+	)
+	(junction
 		(at 85.09 203.2)
 		(diameter 0)
@@
 	)
 	(no_connect
-		(at 165.1 134.62)
+		(at 165.1 135.89)
 	)
 	(no_connect
@@
 	)
 	(no_connect
-		(at 165.1 137.16)
-	)
-	(no_connect
-		(at 165.1 139.7)
-	)
-	(no_connect
-		(at 165.1 144.78)
-	)
-	(no_connect
-		(at 165.1 147.32)
-	)
-	(no_connect
-		(at 165.1 142.24)
+		(at 165.1 138.43)
 	)
 	(no_connect
@@
 	(wire
 		(pts
+			(xy 142.24 106.68) (xy 147.32 106.68)
+		)
+		(stroke
+			(width 0)
+			(type default)
+		)
+	)
+	(wire
+		(pts
 			(xy 104.14 142.24) (xy 119.38 142.24)
 		)
@@
 	(wire
 		(pts
-			(xy 142.24 106.68) (xy 147.32 106.68)
+			(xy 137.16 106.68) (xy 142.24 106.68)
 		)
 		(stroke
@@
 	(wire
 		(pts
-			(xy 137.16 106.68) (xy 142.24 106.68)
-		)
-		(stroke
-			(width 0)
-			(type default)
-		)
-	)
-	(wire
-		(pts
 			(xy 193.04 95.25) (xy 200.66 95.25)
 		)
@@
 	)
 	(symbol
+		(lib_id "Kolibri custom:ESP8685-H4")
+		(at 142.24 132.08 0)
+		(unit 1)
+		(exclude_from_sim no)
+		(in_bom yes)
+		(on_board yes)
+		(dnp no)
+		(fields_autoplaced yes)
+		(property "Reference" "U3"
+			(at 144.3833 157.48 0)
+			(effects
+				(font
+					(size 1.27 1.27)
+				)
+				(justify left)
+			)
+		)
+		(property "Value" "ESP8685-H4"
+			(at 144.3833 160.02 0)
+			(effects
+				(font
+					(size 1.27 1.27)
+				)
+				(justify left)
+			)
+		)
+		(property "Footprint" "Package_DFN_QFN:QFN-28-1EP_4x4mm_P0.4mm_EP2.4x2.4mm"
+			(at 142.748 132.08 0)
+			(effects
+				(font
+					(size 1.27 1.27)
+				)
+				(hide yes)
+			)
+		)
+		(property "Datasheet" "https://www.espressif.com/sites/default/files/documentation/esp32-c3_datasheet_en.pdf"
+			(at 142.748 132.08 0)
+			(effects
+				(font
+					(size 1.27 1.27)
+				)
+				(hide yes)
+			)
+		)
+		(property "Description" "RF Module, ESP32 SoC, RISC-V, WiFi 802.11b/n/g, Bluetooth LE 5, QFN32"
+			(at 142.748 132.08 0)
+			(effects
+				(font
+					(size 1.27 1.27)
+				)
+				(hide yes)
+			)
+		)
+		(pin "25"
+		)
+		(pin "26"
+		)
+		(pin "21"
+		)
+		(pin "16"
+		)
+		(pin "22"
+		)
+		(pin "15"
+		)
+		(pin "14"
+		)
+		(pin "24"
+		)
+		(pin "29"
+		)
+		(pin "12"
+		)
+		(pin "10"
+		)
+		(pin "18"
+		)
+		(pin "2"
+		)
+		(pin "1"
+		)
+		(pin "4"
+		)
+		(pin "7"
+		)
+		(pin "13"
+		)
+		(pin "23"
+		)
+		(pin "27"
+		)
+		(pin "6"
+		)
+		(pin "11"
+		)
+		(pin "28"
+		)
+		(pin "3"
+		)
+		(pin "9"
+		)
+		(pin "5"
+		)
+		(pin "17"
+		)
+		(pin "8"
+		)
+		(pin "20"
+		)
+		(pin "19"
+		)
+		(instances
+			(project ""
+				(path "/1651f454-30c0-48ea-9fcf-6c96a661786a/f86b6c62-cfc0-4383-b218-cc390d004fb8"
+					(reference "U3")
+					(unit 1)
+				)
+			)
+		)
+	)
+	(symbol
 		(lib_id "power:GND")
 		(at 303.53 205.74 0)
@@
 					(unit 1)
 				)
-			)
-		)
-	)
-	(symbol
-		(lib_id "MCU_Espressif:ESP32-C3")
-		(at 142.24 132.08 0)
-		(unit 1)
-		(exclude_from_sim no)
-		(in_bom yes)
-		(on_board yes)
-		(dnp no)
-		(fields_autoplaced yes)
-		(property "Reference" "U3"
-			(at 144.3833 157.48 0)
-			(effects
-				(font
-					(size 1.27 1.27)
-				)
-				(justify left)
-			)
-		)
-		(property "Value" "ESP32-C3"
-			(at 144.3833 160.02 0)
-			(effects
-				(font
-					(size 1.27 1.27)
-				)
-				(justify left)
-			)
-		)
-		(property "Footprint" "Package_DFN_QFN:QFN-32-1EP_5x5mm_P0.5mm_EP3.7x3.7mm"
-			(at 142.748 132.08 0)
-			(effects
-				(font
-					(size 1.27 1.27)
-				)
-				(hide yes)
-			)
-		)
-		(property "Datasheet" "https://www.espressif.com/sites/default/files/documentation/esp32-c3_datasheet_en.pdf"
-			(at 142.748 132.08 0)
-			(effects
-				(font
-					(size 1.27 1.27)
-				)
-				(hide yes)
-			)
-		)
-		(property "Description" "RF Module, ESP32 SoC, RISC-V, WiFi 802.11b/n/g, Bluetooth LE 5, QFN32"
-			(at 142.748 132.08 0)
-			(effects
-				(font
-					(size 1.27 1.27)
-				)
-				(hide yes)
-			)
-		)
-		(pin "5"
-		)
-		(pin "9"
-		)
-		(pin "22"
-		)
-		(pin "15"
-		)
-		(pin "8"
-		)
-		(pin "3"
-		)
-		(pin "6"
-		)
-		(pin "14"
-		)
-		(pin "28"
-		)
-		(pin "2"
-		)
-		(pin "7"
-		)
-		(pin "27"
-		)
-		(pin "30"
-		)
-		(pin "26"
-		)
-		(pin "12"
-		)
-		(pin "33"
-		)
-		(pin "13"
-		)
-		(pin "24"
-		)
-		(pin "29"
-		)
-		(pin "31"
-		)
-		(pin "20"
-		)
-		(pin "11"
-		)
-		(pin "23"
-		)
-		(pin "4"
-		)
-		(pin "32"
-		)
-		(pin "19"
-		)
-		(pin "16"
-		)
-		(pin "25"
-		)
-		(pin "17"
-		)
-		(pin "18"
-		)
-		(pin "10"
-		)
-		(pin "1"
-		)
-		(pin "21"
-		)
-		(instances
-			(project ""
-				(path "/1651f454-30c0-48ea-9fcf-6c96a661786a/f86b6c62-cfc0-4383-b218-cc390d004fb8"
-					(reference "U3")
-					(unit 1)
-				)
