File: Pixel OSD Testboard/Pixel.kicad_sch (KiCad schematic)
At the start: 0 parts

Commit message: wip
Parts:
- added C1, C10, C11, C12, C14, C15, C16, C19, C2, C20, C22, C24, C25, C26, C27, C28, C3, C4, C45, C46, C5, C6, C7, C8, C9: 100n, Capacitor_SMD:C_0402_1005Metric, symbol Device:C
- added C13: 510p, Capacitor_SMD:C_0402_1005Metric, symbol Device:C
- added C17, C18, C47, C51: 10u, Capacitor_SMD:C_0402_1005Metric, symbol Device:C
- added C21, C49, C50: 1u, Capacitor_SMD:C_0402_1005Metric, symbol Device:C
- added C23: 10p, Capacitor_SMD:C_0402_1005Metric, symbol Device:C
- added C29, C30, C31, C32, C33, C34, C35, C36: C, Capacitor_SMD:C_0201_0603Metric, symbol Device:C
- added C37, C38, C39, C40, C41, C42, C43, C44: C, Capacitor_SMD:C_0201_0603Metric_Pad0.64x0.40mm_HandSolder, symbol Device:C
- added C48: 10u, Capacitor_SMD:C_0603_1608Metric, symbol Device:C
- added D1, D4: 1N4148WS, Diode_SMD:D_SOD-323, symbol Diode:1N4148WS
- added D2, D3: ~, Kolibri custom:WS2812B_1615, symbol Kolibri custom:WS2182B_1615
- added D5: SL16, Diode_SMD:D_SOD-123, symbol Device:D
- added J1: USB_C_Receptacle_USB2.0_16P, symbol Connector:USB_C_Receptacle_USB2.0_16P
- added L1: 10u, Inductor_SMD:L_0805_2012Metric, symbol Device:L
- added P1, P2, P3, P4, P5, P6, P7, P8: ~, Kolibri custom:Solder_Pad_rounded, symbol Kolibri custom:Solder_Pad_rounded
- added R1, R2: 5.1k, Resistor_SMD:R_0402_1005Metric, symbol Device:R
- added R10, R12, R14, R19, R20, R32, R33, R8: 100k, Resistor_SMD:R_0402_1005Metric, symbol Device:R
- added R11, R13, R7, R9: 33k, Resistor_SMD:R_0402_1005Metric, symbol Device:R
- added R15, R16, R17, R18, R21, R22, R23, R24, R25, R26, R30, R31: 1k, Resistor_SMD:R_0402_1005Metric, symbol Device:R
- added R27, R36: 10k, Resistor_SMD:R_0402_1005Metric, symbol Device:R
- added R28, R29: 75, Resistor_SMD:R_0402_1005Metric, symbol Device:R
- added R3, R4: 27, Resistor_SMD:R_0402_1005Metric, symbol Device:R
- added R34: 47k, Resistor_SMD:R_0402_1005Metric, symbol Device:R
- added R35: 15k, Resistor_SMD:R_0402_1005Metric, symbol Device:R
- added R5: 680, Resistor_SMD:R_0402_1005Metric, symbol Device:R
- added R6: 620, Resistor_SMD:R_0402_1005Metric, symbol Device:R
- added SW1: ~, Kolibri custom:Button C530669, symbol Kolibri custom:SW_Push w/ GND
- added TP1, TP2, TP3, TP4: TestPoint_Probe, TestPoint:TestPoint_Pad_D1.0mm, symbol Connector:TestPoint_Probe
- added U1: RP2040, Package_DFN_QFN:QFN-56-1EP_7x7mm_P0.4mm_EP3.2x3.2mm, symbol MCU_RaspberryPi:RP2040
- added U2: LM1881, Package_SO:SOIC-8_3.9x4.9mm_P1.27mm, symbol Video:LM1881
- added U3: W25Q16JVSS, Package_SO:SOIC-8_5.3x5.3mm_P1.27mm, symbol Memory_Flash:W25Q16JVSS
- added U4: Opamp_Quad, Package_SO:TSSOP-14_4.4x5mm_P0.65mm, symbol Device:Opamp_Quad
- added U5: 74LVC1G66, Package_TO_SOT_SMD:SOT-353_SC-70-5, symbol 74xGxx:74LVC1G66
- added U6: FSA3157P6X, Package_TO_SOT_SMD:SOT-363_SC-70-6, symbol Analog_Switch:FSA3157P6X
- added U7: TMUX1308DYY, Package_SO:Texas_DYY0016A_TSOT-23-16_2x4.2mm_P0.5mm, symbol Analog_Switch:NMUX1308PW
- added U8: LGS5145, Package_TO_SOT_SMD:SOT-23-6, symbol Regulator_Switching:LGS5145
- added U9: C19631737, Package_TO_SOT_SMD:TO-263-2, symbol Regulator_Linear:MCP1700x-120xxTT
- added Y1: ASE-xxxMHz, Oscillator:Oscillator_SMD_Abracon_ASE-4Pin_3.2x2.5mm_HandSoldering, symbol Oscillator:ASE-xxxMHz
Connections:
- new net: R35.2, R36.1, U8.3 (FB)
- new net: D2.2 (VDD), D3.2 (VDD), D4.1 (K)
- new net: D2.1 (DOUT), D3.4 (DIN)
- new net: R18.1, U5.2
- new net: C46.1, D5.1 (K), L1.1, U8.6 (SW)
- new net: C46.2, U8.1 (BST)
- new net: C23.1, U4.10 (+), U7.3 (Z)
- new net: J1.A5 (CC1), R1.1
- new net: R7.1, U2.1 (CSOUT)
- new net: C12.2, U2.2 (CVIN)
- new net: R9.1, U2.3 (VSOUT)
- new net: R11.1, U2.5 (BPOUT)
- new net: C11.1, R5.1, U2.6 (RSET)
- new net: R13.1, U2.7 (OEOUT)
- new net: R29.1, R30.2, U4.8
- new net: R30.1, R31.2, U4.9 (-)
- new net: U1.20 (XIN), Y1.3 (OUT)
- new net: R21.1, U4.13 (-)
- new net: C35.1, C35.2, C36.1, C36.2
- new net: R15.1, SW1.1
- new net: R15.2, U1.56 (QSPI_SS), U3.1 (~{CS})
- new net: J1.A6 (D+), J1.B6 (D+), R4.1
- new net: J1.A7 (D-), J1.B7 (D-), R3.1
- new net: J1.B5 (CC2), R2.1
- new net: D1.2 (A), U4.1
- new net: R16.1, U4.2 (-)
- new net: C17.1, D1.1 (K), R16.2, R19.1, U6.1
- new net: C21.1, R27.2, U6.3
- new net: U4.5 (+), U6.4
- new net: R34.2, R35.1
- new net: C18.1, R18.2, R20.1, U4.12 (+)
- new net: C12.1, C13.2, R6.2
- new net: R17.1, U4.6 (-)
- new net: C43.1, C43.2, C44.1, C44.2
- new net: U1.55 (QSPI_SD1), U3.2 (DO/IO_{1})
- new net: U1.54 (QSPI_SD2), U3.3 (~{WP}/IO_{2})
- new net: U1.53 (QSPI_SD0), U3.5 (DI/IO_{0})
- new net: U1.52 (QSPI_SCLK), U3.6 (CLK)
- new net: U1.51 (QSPI_SD3), U3.7 (~{HOLD}/~{RESET}/IO_{3})
- new net +10V: C48.1, U8.4 (EN), U8.5 (VIN)
- new net +1V1: C8.1, C9.1, U1.23 (DVDD), U1.45 (VREG_VOUT), U1.50 (DVDD)
- new net +3V3: C1.1, C10.1, C15.1, C2.1, C22.1, C3.1, C4.1, C45.1, C5.1, C50.1, C51.1, C6.1, C7.1, R32.1, U1.1 (IOVDD), U1.10 (IOVDD), U1.22 (IOVDD), U1.26 (RUN), U1.33 (IOVDD), U1.42 (IOVDD), U1.43 (ADC_AVDD), U1.44 (VREG_IN), U1.48 (USB_VDD), U1.49 (IOVDD), U3.8 (VCC), U6.5 (V+), U7.16 (V_{CC}), U9.2 (VO), Y1.1 (EN), Y1.4 (Vdd)
- new net +5V: C14.1, C16.1, C47.1, C49.1, D4.2 (A), J1.A4 (VBUS), J1.A9 (VBUS), J1.B4 (VBUS), J1.B9 (VBUS), L1.2, R34.1, U2.8 (VCC), U4.4 (V+), U9.3 (VI)
- new net BACK_PORCH: R11.2, R12.1, TP3.1, U1.13 (GPIO10)
- new net BLACK_ADC: C19.1, R21.2, R26.2, U1.39 (GPIO27_ADC1), U4.14, U7.14 (Y1)
- new net BLACK_CHG: U1.12 (GPIO9), U5.4
- new net COMPOSITE_SYNC: R7.2, R8.1, TP1.1, U1.5 (GPIO3)
- new net GND: C1.2, C10.2, C11.2, C13.1, C14.2, C15.2, C16.2, C17.2, C18.2, C19.2, C2.2, C20.2, C21.2, C22.2, C23.2, C24.2, C25.2, C26.2, C27.2, C28.2, C3.2, C33.1, C33.2, C34.1, C34.2, C4.2, C41.1, C41.2, C42.1, C42.2, C45.2, C47.2, C48.2, C49.2, C5.2, C50.2, C51.2, C6.2, C7.2, C8.2, C9.2, D2.3 (GND), D3.3 (GND), D5.2 (A), J1.A1 (GND), J1.A12 (GND), J1.B1 (GND), J1.B12 (GND), J1.S1 (SHIELD), R1.2, R10.2, R12.2, R14.2, R19.2, R2.2, R20.2, R28.2, R31.1, R33.2, R36.2, R5.2, R8.2, SW1.2, SW1.3 (MP), SW1.4 (MP), U1.19 (TESTEN), U1.57 (GND), U2.4 (GND), U3.4 (GND), U4.11 (V-), U6.2 (GND), U7.4 (Y7), U7.6 (~{E}), U7.8 (GND), U8.2 (GND), U9.1 (GND), Y1.2 (GND)
- new net GREY1: C27.1, R25.2, R26.1, U7.15 (Y2)
- new net GREY2: C26.1, R24.2, R25.1, U7.12 (Y3)
- new net GREY3: C25.1, R23.2, R24.1, U7.1 (Y4)
- new net GREY4: C24.1, R22.2, R23.1, U7.5 (Y5)
- new net LED: D2.4 (DIN), U1.2 (GPIO0)
- new net ODD_FRAME: R13.2, R14.1, TP4.1, U1.7 (GPIO5)
- new net RX0: P4.1, U1.16 (GPIO13)
- new net RX1: P8.1, U1.32 (GPIO21)
- new net SWCLK: P5.1, U1.24 (SWCLK)
- new net SWDIO: P6.1, U1.25 (SWD)
- new net TEST_ADC: C28.1, R32.2, R33.1, U1.40 (GPIO28_ADC2)
- new net TX0: P3.1, U1.15 (GPIO12)
- new net TX1: P7.1, U1.31 (GPIO20)
- new net USBD+: R4.2, U1.47 (USB_DP)
- new net USBD-: R3.2, U1.46 (USB_DM)
- new net VIDEO_IN: P1.1, R28.1, R6.1, U4.3 (+), U5.1, U7.13 (Y0)
- new net VIDEO_OUT: P2.1, R29.2
- new net VSEL0: U1.8 (GPIO6), U7.11 (S0)
- new net VSEL1: U1.9 (GPIO7), U7.10 (S1)
- new net VSEL2: U1.11 (GPIO8), U7.9 (S2)
- new net VSYNC: R10.1, R9.2, TP2.1, U1.6 (GPIO4)
- new net VWHITE_PWM: R27.1, U1.3 (GPIO1)
- new net WHITE_ADC: C20.1, R17.2, R22.1, U1.38 (GPIO26_ADC0), U4.7, U7.2 (Y6)
- new net WHITE_SELECT: U1.4 (GPIO2), U6.6
- no-connect marks 0 -> 20
Other:
- note added: "ADC Test Test whether a buffer opamp is actually needed, once a filter cap exists"
- note added: "C285963"
- note added: "Extract Sync, the rest is technically optional"
- note added: "Soldering Tests Test whether it is possible to hand place 0201 components, test using different copper heat sinks Top row: regular 0201 footprint Bottom row: handsolder footprint"
- note added: "Use Sync/Back Porch to get black intervals Use Peak detector to get white level, or PWM + RC LPF to create white level Use buffers to copy those levels, use resistor ladder to create grey levels"
- note added: "Use analog MUX to combine the signals into one, pixel by pixel"

Commit message: Update Pixel.kicad_sch
Parts:
- removed D2, D3: ~, Kolibri custom:WS2812B_1615, symbol Kolibri custom:WS2182B_1615
- removed D4: 1N4148WS, Diode_SMD:D_SOD-323, symbol Diode:1N4148WS
- added D2: yellow, LED_SMD:LED_0603_1608Metric, symbol Device:LED
- added D3: green, LED_SMD:LED_0603_1608Metric, symbol Device:LED
- added D4: red, LED_SMD:LED_0603_1608Metric, symbol Device:LED
- added P10, P11, P12, P13, P14, P9: ~, Kolibri custom:Solder_Pad_octa, symbol Kolibri custom:Solder_Pad_octa
- added P15, P16, P17, P18: ~, Kolibri custom:Solder_Pad_rect, symbol Kolibri custom:Solder_Pad_rect
- added R37, R38: 470, Resistor_SMD:R_0402_1005Metric, symbol Device:R
- added R39: 1k, Resistor_SMD:R_0402_1005Metric, symbol Device:R
- added TP5, TP6, TP7, TP8: TestPoint_Probe, TestPoint:TestPoint_Pad_D1.0mm, symbol Connector:TestPoint_Probe
Connections:
- net +10V: now also P13.1, P14.1
- net +3V3: now also P11.1, P9.1, R39.1
- net +5V: now also P10.1, P12.1
- net BLACK_ADC: now also TP8.1
- net GND: now also D2.1 (K), D3.1 (K), D4.1 (K), P15.1, P16.1, P17.1, P18.1
- net WHITE_ADC: now also TP7.1
- net at C17.1, D1.1 (K), R16.2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: now also TP5.1
- net at C21.1, R27.2, U6.3: now also TP6.1
- net LED1: now reaches U1.18 (GPIO15)
- net LED1: now also R38.1
- net LED2: now reaches U1.27 (GPIO16)
- net LED2: now also R37.1
- net LED: no longer names the net of U1.2 (GPIO0)
- new net: D4.2 (A), R39.2
- new net: D2.2 (A), R38.2
- new net: D3.2 (A), R37.2
- no-connect marks 20 -> 19
Other:
- note added: "3.3V LDO, 200mA"
- note added: "5V DCDC, 400mA (inductor limited), 1.2MHz"
- moved on the sheet: C49, C50, C51, U9

Commit message: wip
Parts:
- removed R17, R21, R30, R31: 1k, Resistor_SMD:R_0402_1005Metric, symbol Device:R
- added C52: 10u, Capacitor_SMD:C_0603_1608Metric_Pad1.08x0.95mm_HandSolder, symbol Device:C
- added C53: 1u, Capacitor_SMD:C_0603_1608Metric_Pad1.08x0.95mm_HandSolder, symbol Device:C
- added C54: 100n, Capacitor_SMD:C_0402_1005Metric, symbol Device:C
- added C55: 1u, Capacitor_SMD:C_0402_1005Metric, symbol Device:C
- added Q1: 2SK3019, Package_TO_SOT_SMD:SOT-523, symbol Transistor_FET:2SK3019
- added R40: 1M, Resistor_SMD:R_0603_1608Metric_Pad0.98x0.95mm_HandSolder, symbol Device:R
- added R41: 2.2M, Resistor_SMD:R_0603_1608Metric_Pad0.98x0.95mm_HandSolder, symbol Device:R
- added R42: 390k, Resistor_SMD:R_0603_1608Metric_Pad0.98x0.95mm_HandSolder, symbol Device:R
- added R43, R44: 1k, Resistor_SMD:R_0603_1608Metric_Pad0.98x0.95mm_HandSolder, symbol Device:R
- added TP10, TP9: TestPoint_Probe, TestPoint:TestPoint_Pad_D1.0mm, symbol Connector:TestPoint_Probe
- added U10: FSA3157P6X, Package_TO_SOT_SMD:SOT-363_SC-70-6, symbol Analog_Switch:FSA3157P6X
- added U11: Opamp_Quad, Package_SO:TSSOP-14_4.4x5mm_P0.65mm, symbol Device:Opamp_Quad
- C11, C12, C13, C17, C18: footprint Capacitor_SMD:C_0402_1005Metric -> Capacitor_SMD:C_0603_1608Metric_Pad1.08x0.95mm_HandSolder
- C23, C24, C25, C26, C27: footprint Capacitor_SMD:C_0402_1005Metric -> Capacitor_SMD:C_0402_1005Metric_Pad0.74x0.62mm_HandSolder
- J1: footprint (none) -> Kolibri custom:USB-C SMD+THT
- R10, R11, R12, R13, R14, R7, R8, R9: footprint Resistor_SMD:R_0402_1005Metric -> Resistor_SMD:R_0402_1005Metric_Pad0.72x0.64mm_HandSolder
- R16: value 1k -> 10k
- R18: value 1k -> 100; footprint Resistor_SMD:R_0402_1005Metric -> Resistor_SMD:R_0603_1608Metric_Pad0.98x0.95mm_HandSolder
- R19, R20, R22, R23, R24, R25, R26, R5, R6: footprint Resistor_SMD:R_0402_1005Metric -> Resistor_SMD:R_0603_1608Metric_Pad0.98x0.95mm_HandSolder
- U9: footprint Package_TO_SOT_SMD:TO-263-2 -> Package_TO_SOT_SMD:SOT-23-3
Connections:
- net +3V3: now also R40.1, R41.1
- net +5V: now also C54.1, U11.4 (V+)
- net BLACK_ADC: now also U4.13 (-)
- net GND: now also C54.2, C55.2, Q1.2 (S), R42.2, R44.2, U11.11 (V-)
- net VIDEO_IN: now also C53.1; no longer U4.3 (+), U5.1, U7.13 (Y0)
- net WHITE_ADC: now also U4.6 (-)
- net WHITE_SAH: now reaches C17.1, D1.1 (K), R19.1, TP5.1, U6.1
- net WHITE_SAH: now also U4.2 (-); no longer R16.2
- net at U4.8: now also U4.9 (-), C52.1; no longer R29.1
- net VBLACK_PWM: now reaches R16.1
- net VBLACK_PWM: now also U1.29 (GPIO18); no longer U4.2 (-)
- net BLACK_SAH: now reaches C18.1, R18.2, R20.1
- net BLACK_SAH: now also R40.2, U10.1; no longer U4.12 (+)
- net SYNC_CLAMP: now reaches U1.14 (GPIO11)
- net SYNC_CLAMP: now also Q1.1 (G)
- net BLACK_SELECT: now reaches U1.28 (GPIO17)
- net BLACK_SELECT: now also U10.6
- new net: C53.2, Q1.3 (D), R41.2, R42.1, U11.3 (+)
- new net: C52.2, R29.1
- new net: R43.2, R44.1, U11.2 (-)
- new net: C55.1, R16.2, TP10.1, U10.3
- new net: U10.4, U4.12 (+)
- new net VIDEO_IN_CLAMP: R43.1, TP9.1, U11.1, U4.3 (+), U5.1, U7.13 (Y0)
- no-connect marks 19 -> 28
Other:
- note added: "Input stage AC-couple, then tie to ground during sync. Buffer opamp for low impedance output"
- note added: "Solder Pads"
- note added: "Use Sync/Back Porch to get black intervals (sample and hold, SAH) Use Peak detector to get white level, or PWM + RC LPF to create white level Use buffers to copy those levels, use resistor ladder to create grey levels"
- note added: "Voltage regulators"
- note removed: "Use Sync/Back Porch to get black intervals Use Peak detector to get white level, or PWM + RC LPF to create white level Use buffers to copy those levels, use resistor ladder to create grey levels"
- moved on the sheet: C1, C10, C11, C12, C13, C14, C15, C16, C18, C19, C2, C22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

Commit message: ^wip layout
Parts:
- removed TP7: TestPoint_Probe, TestPoint:TestPoint_Pad_D1.0mm, symbol Connector:TestPoint_Probe
- removed U11: Opamp_Quad, Package_SO:TSSOP-14_4.4x5mm_P0.65mm, symbol Device:Opamp_Quad
- added U11: OPA188xxDBV, Package_TO_SOT_SMD:TSOT-23-5, symbol Amplifier_Operational:OPA188xxDBV
Connections:
- net +5V: now also U11.5 (V+)
- net BLACK_ADC: no longer TP8.1
- net BLACK_SAH: now also TP8.1
- net GND: now also U11.2 (V-)
- net VIDEO_IN_CLAMP: now also U11.1
- net at C53.2, Q1.3 (D), R41.2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: now also U11.3 (+)
- net at R43.2, R44.1: now also U11.4 (-)
- no-connect marks 28 -> 19
Other:
- moved on the sheet: C54, R44, TP8

Commit message: 0 DRC errors
Parts:
- added C56, C57: 100n, Capacitor_SMD:C_0402_1005Metric, symbol Device:C
- added unit 2 of U10
- added unit 2 of U5
Connections:
- net +3V3: now also C56.1, C57.1, U10.5 (V+), U5.5 (VCC)
- net GND: now also C56.2, C57.2, U10.2 (GND), U5.3 (GND)
- net LED1: now also U1.27 (GPIO16); no longer U1.18 (GPIO15)
- net LED2: now also U1.18 (GPIO15); no longer U1.27 (GPIO16)
- net VWHITE_PWM: now also U1.36 (GPIO24); no longer U1.3 (GPIO1)
- net WHITE_SELECT: now also U1.37 (GPIO25); no longer U1.4 (GPIO2)
- no-connect marks 19 -> 29
